File: SP Block/input_conditioning_r2.kicad_sch (KiCad schematic)
At the start: 11 parts, among them J1 Conn_Coaxial, J2 Conn_Coaxial, J3 Conn_01x02_Socket, J4 Conn_01x02_Socket

Commit message: Refactor and polishing
Parts:
- C19: footprint (none) -> Capacitor_THT:C_Radial_D5.0mm_H11.0mm_P2.00mm
- C2, C3: value 1u -> 5u; footprint (none) -> Capacitor_THT:C_Radial_D5.0mm_H11.0mm_P2.00mm
Other:
- removed sheet RP2040
- note removed: "??"
- moved on the sheet: J4
Changed lines of the file:
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@@
 		)
 	)
-	(text "??"
-		(exclude_from_sim no)
-		(at 26.67 47.752 0)
-		(effects
-			(font
-				(size 2.54 2.54)
-				(thickness 0.254)
-				(bold yes)
-			)
-		)
-	)
 	(text "aluminum"
 		(exclude_from_sim no)
@@
 		)
 	)
+	(text "aluminum"
+		(exclude_from_sim no)
+		(at 29.21 48.514 0)
+		(effects
+			(font
+				(size 1.27 1.27)
+			)
+		)
+	)
 	(text "ADC Drivers"
 		(exclude_from_sim no)
@@
 		)
 	)
-	(text "??"
+	(text "Power\n(ground probe to 0V)"
 		(exclude_from_sim no)
-		(at 34.036 56.388 0)
+		(at 124.968 134.366 0)
 		(effects
 			(font
-				(size 2.54 2.54)
+				(size 3.81 3.81)
 				(thickness 0.254)
 				(bold yes)
@@
 		)
 	)
-	(text "Power\n(ground probe to 0V)"
+	(text "aluminum"
 		(exclude_from_sim no)
-		(at 124.968 134.366 0)
+		(at 30.988 59.436 0)
 		(effects
 			(font
-				(size 3.81 3.81)
-				(thickness 0.254)
-				(bold yes)
+				(size 1.27 1.27)
 			)
 		)
@@
 	(wire
 		(pts
-			(xy 229.87 57.15) (xy 238.76 57.15)
+			(xy 240.03 50.8) (xy 248.92 50.8)
 		)
 		(stroke
@@
 	(wire
 		(pts
-			(xy 91.44 114.3) (xy 114.3 114.3)
-		)
-		(stroke
-			(width 0)
-			(type default)
-		)
-	)
-	(wire
-		(pts
 			(xy 17.78 43.18) (xy 17.78 38.1)
 		)
@@
 	(wire
 		(pts
+			(xy 91.44 114.3) (xy 114.3 114.3)
+		)
+		(stroke
+			(width 0)
+			(type default)
+		)
+	)
+	(wire
+		(pts
 			(xy 59.69 121.92) (xy 46.99 121.92)
 		)
@@
 	(wire
 		(pts
-			(xy 229.87 59.69) (xy 238.76 59.69)
+			(xy 240.03 53.34) (xy 248.92 53.34)
 		)
 		(stroke
@@
 	)
 	(label "output_1"
-		(at 229.87 57.15 0)
+		(at 240.03 50.8 0)
 		(effects
 			(font
@@
 	)
 	(label "output_2"
-		(at 229.87 59.69 0)
+		(at 240.03 53.34 0)
 		(effects
 			(font
@@
 			)
 		)
-		(property "Value" "1u"
+		(property "Value" "5u"
 			(at 29.21 57.1499 0)
 			(effects
@@
 			)
 		)
-		(property "Footprint" ""
+		(property "Footprint" "Capacitor_THT:C_Radial_D5.0mm_H11.0mm_P2.00mm"
 			(at 26.3652 59.69 0)
 			(effects
@@
 			)
 		)
-		(property "Value" "1u"
+		(property "Value" "5u"
 			(at 21.59 48.2599 0)
 			(effects
@@
 			)
 		)
-		(property "Footprint" ""
+		(property "Footprint" "Capacitor_THT:C_Radial_D5.0mm_H11.0mm_P2.00mm"
 			(at 18.7452 50.8 0)
 			(effects
@@
 			)
 		)
-		(property "Footprint" ""
+		(property "Footprint" "Capacitor_THT:C_Radial_D5.0mm_H11.0mm_P2.00mm"
 			(at 115.2652 124.46 0)
 			(effects
@@
 	(symbol
 		(lib_id "Connector:Conn_01x02_Socket")
-		(at 243.84 57.15 0)
+		(at 254 50.8 0)
 		(unit 1)
 		(exclude_from_sim yes)
@@
 		(fields_autoplaced yes)
 		(property "Reference" "J4"
-			(at 245.11 57.1499 0)
+			(at 255.27 50.7999 0)
 			(effects
 				(font
@@
 		)
 		(property "Value" "Conn_01x02_Socket"
-			(at 245.11 59.6899 0)
+			(at 255.27 53.3399 0)
 			(effects
 				(font
@@
 		)
 		(property "Footprint" ""
-			(at 243.84 57.15 0)
+			(at 254 50.8 0)
 			(effects
 				(font
@@
 		)
 		(property "Datasheet" "~"
-			(at 243.84 57.15 0)
+			(at 254 50.8 0)
 			(effects
 				(font
@@
 		)
 		(property "Description" "Generic connector, single row, 01x02, script generated"
-			(at 243.84 57.15 0)
+			(at 254 50.8 0)
 			(effects
 				(font
@@
 				)
 			)
-		)
-	)
-	(sheet
-		(at 224.79 21.59)
-		(size 39.37 22.86)
-		(exclude_from_sim yes)
-		(in_bom no)
-		(on_board no)
-		(dnp no)
-		(fields_autoplaced yes)
-		(stroke
-			(width 0.1524)
-			(type solid)
-		)
-		(fill
-			(color 0 0 0 0.0000)
-		)
-		(property "Sheetname" "RP2040"
-			(at 224.79 20.8784 0)
-			(effects
-				(font
-					(size 1.27 1.27)
-				)
-				(justify left bottom)
-			)
-		)
-		(property "Sheetfile" "RP2040.kicad_sch"
-			(at 224.79 45.0346 0)
-			(effects
-				(font
-					(size 1.27 1.27)
-				)
-				(justify left top)
-			)
-		)
-		(instances
-			(project "input_conditioning_r2"
-				(path "/e8001732-a560-4bb6-87d1-5a7552612e81"
-					(page "3")
-				)
-			)

Commit message: updated with available part sizes
Parts:
- C2, C3: value 5u -> 1u
Changed lines of the file:
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@@
 			)
 		)
-		(property "Value" "5u"
+		(property "Value" "1u"
 			(at 29.21 57.1499 0)
 			(effects
@@
 			)
 		)
-		(property "Value" "5u"
+		(property "Value" "1u"
 			(at 21.59 48.2599 0)
 			(effects
