File: SP Block/real_signal_processing.kicad_sch (KiCad schematic)
At the start: 15 parts, among them U1 OPA2365AID

Commit message: Refactor and polishing
Parts:
- added C34, C36: 100n, symbol Device:C
- C20: footprint (none) -> Capacitor_THT:C_Rect_L7.0mm_W4.5mm_P5.00mm
- U1: footprint D8 -> OPA2365:D8
Connections:
- net +5V: now also C34.1, C36.1
- net GND: now also C34.2, C36.2
Other:
- note added: "C0G"
- note added: "X7R 50V"
- note added: "X7R OPA INA+"
- note added: "X7R OPA INB+"
- note added: "X7R OPA V+"
- note removed: "1.25Vpp"
- note removed: "2.5Vpp"
- note removed: "5Vpp"
- note removed: "??"
- note removed: "Ceramic"
- note removed: "Electrolytic"
- moved on the sheet: C21, U1

Commit message: updated with available part sizes
Parts:
- removed D5, D6: 1N4617, symbol Device:D
- added C38: 100n, symbol Device:C
- added D3, D5: 1N4148, Diode_THT:D_DO-35_SOD27_P7.62mm_Horizontal, symbol Diode:1N4148
- C26: value 500p -> 680p
- C27: value 5p -> 20p
- C29: value 10p -> 33p
- R18, R19, R26: value 50k -> 47k
Connections:
- net +5V: now also C38.1, D3.1 (K)
- net GND: now also C38.2, D5.2 (A)
- new net: D3.2 (A), D5.1 (K)
Other:
- note added: "X7R OPA V-"
