File: PCB schematic/signal_processing.kicad_sch (KiCad schematic)
At the start: 19 parts, among them U3 OPA365xxD, U6 OPA365xxD

Commit message: pcb initial complete revision
Connections:
- net ac_coupled: now also D1.1 (K), D9.2 (A)
Changed lines of the file:
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@@
+	)
+	(junction
+		(at 83.82 110.49)
+		(diameter 0)
+		(color 0 0 0 0)
 	)
 	(junction
@@
 	(wire
 		(pts
+			(xy 83.82 110.49) (xy 83.82 113.03)
+		)
+		(stroke
+			(width 0)
+			(type default)
+		)
+	)
+	(wire
+		(pts
 			(xy 198.12 85.09) (xy 198.12 105.41)
 		)
@@
 	(wire
 		(pts
+			(xy 83.82 110.49) (xy 92.71 110.49)
+		)
+		(stroke
+			(width 0)
+			(type default)
+		)
+	)
+	(wire
+		(pts
 			(xy 119.38 97.79) (xy 121.92 97.79)
 		)
@@
 	(wire
 		(pts
-			(xy 74.93 110.49) (xy 92.71 110.49)
+			(xy 74.93 110.49) (xy 83.82 110.49)
 		)
 		(stroke
@@
 	(wire
 		(pts
-			(xy 83.82 107.95) (xy 83.82 113.03)
-		)
-		(stroke
+			(xy 83.82 107.95) (xy 83.82 110.49)
+		)
+		(stroke
